Commit message: Add constrained planning tests

File: manipulation_pipeline_tests/urdf/single_ur.urdf.xacro (robot description, xacro)
@@ -3,5 +3,40 @@
     <xacro:include filename="$(find manipulation_pipeline_tests)/urdf/ur_simple.urdf.xacro" />
     <xacro:include filename="$(find ur_description)/urdf/ros2_control_mock_hardware.xacro" />
+    <material name="red">
+        <color rgba="1 0 0 0.2" />
+    </material>
     <link name="world" />
     <xacro:ur_simple name="ur" ur_type="ur10e" parent="world" />
+    <xacro:macro name="collision_box" params="name parent length width height *origin">
+        <link name="${name}">
+            <visual>
+                <geometry>
+                    <box size="${length} ${width} ${height}" />
+                </geometry>
+                <material name="red" />
+            </visual>
+            <collision>
+                <geometry>
+                    <box size="${length} ${width} ${height}" />
+                </geometry>
+            </collision>
+        </link>
+        <joint name="${name}_joint" type="fixed">
+            <parent link="${parent}" />
+            <child link="${name}" />
+            <xacro:insert_block name="origin" />
+        </joint>
+    </xacro:macro>
+    <xacro:collision_box name="floor" parent="world" length="2.0" width="2.0" height="0.1">
+        <origin xyz="0 0 -0.05" />
+    </xacro:collision_box>
+    <xacro:collision_box name="box_1" parent="world" length="0.5" width="0.1" height="0.8">
+        <origin xyz="0.6 0.4 0.4" />
+    </xacro:collision_box>
+    <xacro:collision_box name="box_2" parent="world" length="0.5" width="0.1" height="0.8">
+        <origin xyz="0.6 -0.4 0.4" />
+    </xacro:collision_box>
+    <xacro:collision_box name="box_3" parent="world" length="0.5" width="0.1" height="0.8">
+        <origin xyz="-0.6 0 0.4" rpy="0 0 ${pi}" />
+    </xacro:collision_box>
 </robot>
